File: 3DPCB_4L.kicad_sch (KiCad schematic)
At the start: 204 parts, among them IC1 A5984_LP, IC2 A5984_LP, IC3 A5984_LP, IC4 A5984_LP, IC5 A5984_LP, IC6 MP9943, J10 , J11 , J12 , J13 , J14 , J15 , J16 , J2 , J3 , J4 , J5 , J6 , J7 , J8 , J9 , K1 CONN_3, K2 CONN_3, K3 CONN_3, K4 CONN_3, K5 CONN_3, K6 CONN_3, K7 CONN_3, K8 CONN_3, K9 CONN_3, P1 CONN_8, P11 CONN_3X2, P12 CONN_3X2, P13 CONN_4, P2 CONN_8, P3 CONN_01X02, P5 CONN_4, P6 CONN_4, P7 CONN_4, P8 CONN_02X03, P9 CONN_4, U1 CONN_4_LERCHE, U10 MICRO-SD, U11 TC4427, U12 MCP4728, U13 CONN_4_LERCHE, U15 SPST_MOMENTARY, U16 CONN_4_LERCHE, U2 SPST_MOMENTARY, U21 CONN_4_LERCHE, U22 CONN_4_LERCHE, U23 MCP4728, U24 IRFH5302, U25 CONN_4_LERCHE, U3 BSS84, U4 CONN_4_LERCHE, U5 IRFH5302, U6 LPC1768_TQFP100, U7 IRFH5302, U8 IRFH5302, U9 TC4427

Commit message: Updated with KiCAD 6.0.4
Parts:
- 12MHz1: renamed from OSC1; value QX2 -> (none); footprint LercheTech:Lerche_Oscillator_2.5x2.0mm -> (none)
- C1, C12, C13, C14, C15, C16, C17, C19, C2, C20, C21, C22, C23, C28, C29, C30, C31, C32, C33, C34, C35, C39, C44, C45, C46, C47, C50, C51, C52, C53, C54, C6, C64, C65, C67, C69, C71: value 100n -> (none)
- C10, C3, C4, C7: value 10uF -> (none)
- C11, C24, C25, C26, C27, C70: value 100uF -> (none)
- C18: value 100pF -> (none)
- C36, C37, C8: value 100nF -> (none)
- C38: value 10n -> (none)
- C40, C41, C42, C48, C55: value 220n -> (none)
- C43: value 47uF -> (none)
- C49: value 1uF -> (none)
- C5, C9: value 18p -> (none)
- D5: value DIODESCH -> (none)
- D6, D7, D8: value LED -> (none)
Connections:
- net GND: now also C1.2, R14.2
- net ~{RESET}: now also C1.1

Commit message: Minor changes
Parts:
- C1, C12, C13, C14, C15, C16, C17, C18, C19, C2, C20, C21, C22, C23, C28, C29, C30, C31, C32, C33, C34, C35, C36, C37, C38, C39, C40, C41, C42, C44, C45, C46, C47, C48, C49, C5, C50, C51, C52, C53, C54, C55, C6, C64, C65, C67, C69, C71, C8, C9: footprint Capacitor_SMD:C_0603_1608Metric -> (none)
- C10, C3, C4, C7: footprint Capacitors_Tantalum_SMD:TantalC_SizeA_EIA-3216_Reflow -> (none)
- C11, C24, C25, C26, C27, C70: footprint Capacitor_THT:CP_Radial_D6.3mm_P2.50mm -> (none)
- C43: footprint Capacitor_SMD:CP_Elec_5x5.8 -> (none)
- C56, C57: value np -> (none); footprint Capacitor_SMD:C_0603_1608Metric -> (none)
- CONN1: value USB_MINI -> (none); footprint Connector_USB:USB_Micro-B_Molex-105017-0001 -> (none)
- D1, D11, D12, D13, D14, D2, D3, D4: value LED -> (none); footprint LED_SMD:LED_0603_1608Metric -> (none)
- D10: value Vz10V/0.5W -> (none); footprint Diodes_SMD:SMA_Standard -> (none)
- D5: footprint Diode_SMD:D_SOD-323 -> (none)
- D6, D7, D8: footprint LED_SMD:LED_0603_1608Metric -> (none)
- D9: value DIODESCH -> (none); footprint Diode_SMD:D_SOD-323 -> (none)
- FID1, FID2, FID3, FID4: value FIDUCIAL -> (none); footprint LercheTech:Lerche_Fiducial -> (none)
- IC1, IC2, IC3, IC4, IC5: value A5984_LP -> (none); footprint Package_SO:TSSOP-24-1EP_4.4x7.8mm_P0.65mm_EP3.2x5mm -> (none)
- IC6: value MP9943 -> (none); footprint LercheTech:Lerche_MP9943 -> (none)
- J10, J11, J12, J13, J14, J15, J16, J2, J3, J4, J5, J6, J7, J8, J9: value (none) -> (none); footprint LercheTech:Lerche_2PsolderJumper -> (none)
- K1, K2, K3, K4, K5, K6, K8, K9: value CONN_3 -> (none); footprint Connector_PinHeader_2.54mm:PinHeader_1x03_P2.54mm_Vertical -> (none)
- K7: value CONN_3 -> (none); footprint Connector_PinHeader_1.27mm:PinHeader_1x03_P1.27mm_Vertical -> (none)
- L1: value INDUCTOR -> (none); footprint Inductor_SMD:L_0603_1608Metric -> (none)
- L2: value IHLP1212BZER2R2M11 -> (none); footprint LercheTech:Lerche_IHLP-1212BZ-11_Inductor -> (none)
- P1: value CONN_8 -> (none); footprint Connector_PinSocket_2.54mm:PinSocket_1x08_P2.54mm_Vertical -> (none)
- P11: value CONN_3X2 -> (none); footprint Connector_PinSocket_2.54mm:PinSocket_2x03_P2.54mm_Vertical -> (none)
- P12: value CONN_3X2 -> (none); footprint LercheTech:Lerche_6P_1.6mm_2ROW -> (none)
- P13, P5, P6, P7, P9: value CONN_4 -> (none); footprint Connector_PinSocket_2.54mm:PinSocket_1x04_P2.54mm_Vertical -> (none)
- P2: value CONN_8 -> (none); footprint LercheTech:Lerche_8P_CONN_3,5mm -> (none)
- P3: value CONN_01X02 -> (none); footprint Connector_PinSocket_2.54mm:PinSocket_1x02_P2.54mm_Vertical -> (none)
- P8: value CONN_02X03 -> (none); footprint LercheTech:Lerche_Molex_Microfit_0430450607 -> (none)
- R1, R18, R19, R27, R41, R42, R43, R9: value 10k -> (none); footprint Resistor_SMD:R_0603_1608Metric -> (none)
- R10, R12, R13, R34: value 4K7 -> (none); footprint Resistor_SMD:R_0603_1608Metric -> (none)
- R11: value 1k5 -> (none); footprint Resistor_SMD:R_0603_1608Metric -> (none)
- R14, R15, R16, R20: value 47k -> (none); footprint Resistor_SMD:R_0603_1608Metric -> (none)
- R17: value 1k -> (none); footprint Resistor_SMD:R_0805_2012Metric -> (none)
- R2, R28, R3, R4, R5, R6: value 1k -> (none); footprint Resistor_SMD:R_0603_1608Metric -> (none)
- R21, R22, R23, R24, R29, R30, R31, R32, R33, R37: value 0R05 -> (none); footprint Resistor_SMD:R_1206_3216Metric -> (none)
- R25, R26, R46, R47, R48: value 0R -> (none); footprint Resistor_SMD:R_0603_1608Metric -> (none)
- R35: value 1M -> (none); footprint Resistor_SMD:R_0603_1608Metric -> (none)
- R36: value 20R -> (none); footprint Resistor_SMD:R_0603_1608Metric -> (none)
- R38: value 51k -> (none); footprint Resistor_SMD:R_0603_1608Metric -> (none)
- R39: value 13k -> (none); footprint Resistor_SMD:R_0603_1608Metric -> (none)
- R40: value 41k2 -> (none); footprint Resistor_SMD:R_0603_1608Metric -> (none)
- R44, R45: value 3k3 -> (none); footprint Resistor_SMD:R_0603_1608Metric -> (none)
- R49, R50, R51, R52: value 4k7 -> (none); footprint Resistor_SMD:R_0603_1608Metric -> (none)
- R53: value 100R -> (none); footprint Resistor_SMD:R_0603_1608Metric -> (none)
- R55: value 5k8 -> (none); footprint Resistor_SMD:R_0603_1608Metric -> (none)
- R56, R57, R58, R59: value 10R -> (none); footprint Resistor_SMD:R_0603_1608Metric -> (none)
- R7, R8: value 33R -> (none); footprint Resistor_SMD:R_0603_1608Metric -> (none)
- U1, U13, U16, U21, U22, U25, U4: value CONN_4_LERCHE -> (none); footprint Connector_PinSocket_2.54mm:PinSocket_1x04_P2.54mm_Vertical -> (none)
- U10: value MICRO-SD -> (none); footprint LercheTech:Lerche_Molex_502774-0891 -> (none)
- U11, U9: value TC4427 -> (none); footprint SMD_Packages:SOIC-8-N -> (none)
- U12, U23: value MCP4728 -> (none); footprint LercheTech:Lerche_MSOP-10 -> (none)
- U15, U2: value SPST_MOMENTARY -> (none); footprint LercheTech:Lerche_SPST_ITEAD -> (none)
- U24, U5, U7, U8: value IRFH5302 -> (none); footprint LercheTech:Lerche_PQFN_5x6B -> (none)
- U3: value BSS84 -> (none); footprint Package_TO_SOT_SMD:SOT-23 -> (none)
- U6: value LPC1768_TQFP100 -> (none); footprint Housings_QFP:TQFP-100_14x14mm_Pitch0.5mm -> (none)
